File: Hardware/AquaTimer.kicad_pcb (KiCad board)
At the start: 2 copper layers, 4 parts, among them J1 Conn_01x03

Commit message: Add files via upload
Parts:
- added J2: Conn_01x03, Connector_PinHeader_2.54mm:PinHeader_1x03_P2.54mm_Vertical, F.Cu at (148.0, 105.5)
- added J3: Screw_Terminal_01x02, TerminalBlock:TerminalBlock_MaiXu_MX126-5.0-02P_1x02_P5.00mm, F.Cu at (137.5, 105.5)
- added R2: 330, Resistor_THT:R_Axial_DIN0207_L6.3mm_D2.5mm_P10.16mm_Horizontal, F.Cu at (168.1, 121.0)
- added U1: L7805, L7805:TO255P1020X450X2000-3, F.Cu at (145.4, 99.0)
Connections:
- A1 pad 15: unconnected-(A1-GPIO11-Pad15) -> Net-(A1-GPIO11)
- A1 pad 37: unconnected-(A1-3V3_EN-Pad37) -> +3,3V
- A1 pad 39: unconnected-(A1-VSYS-Pad39) -> +5V
Routing:
- net +5V: track 41.6 -> 145.6 mm
- net +3,3V: track 0.00 -> 100.6 mm
- net Net-(A1-GPIO11): track 0.00 -> 49.5 mm
- net Net-(J3-Pin_1): track 0.00 -> 10.7 mm
