File: Hardware/AquaTimer.kicad_sch (KiCad schematic)
At the start: 4 parts, among them J1 Conn_01x03

Commit message: Add files via upload
Parts:
- added J2: Conn_01x03, Connector_PinHeader_2.54mm:PinHeader_1x03_P2.54mm_Vertical, symbol Connector_Generic:Conn_01x03
- added J3: Screw_Terminal_01x02, TerminalBlock:TerminalBlock_MaiXu_MX126-5.0-02P_1x02_P5.00mm, symbol Connector:Screw_Terminal_01x02
- added R2: 330, Resistor_THT:R_Axial_DIN0207_L6.3mm_D2.5mm_P10.16mm_Horizontal, symbol Device:R
- added U1: L7805, L7805:TO255P1020X450X2000-3, symbol Regulator_Linear:L7805
Connections:
- net +5V: now also A1.39 (VSYS), J2.1 (Pin_1), U1.3 (OUT)
- net GND: now also J2.3 (Pin_3), J3.2 (Pin_2), U1.2 (GND)
- net at A1.15 (GPIO11): now also J2.2 (Pin_2), R2.2
- net +3,3V: now reaches A1.37 (3V3_EN)
- net +3,3V: now also R2.1
- new net: J3.1 (Pin_1), U1.1 (IN)
